Commit message: color update

File: install/my_robot_description/share/my_robot_description/urdf/amr_robot.urdf.xacro (robot description, xacro)
@@ -1,4 +1,14 @@
 <?xml version="1.0"?>
 <robot name="amr_robot" xmlns:xacro="http://ros.org/wiki/xacro">
+    <!-- Materials -->
+  <material name="black">
+    <color rgba="0.2 0.2 0.2 1"/>
+  </material>
+  <material name="gray">
+    <color rgba="0.5 0.5 0.5 1"/>
+  </material>
+  <material name="red">
+    <color rgba="1 0 0 1"/>
+  </material>
   <!-- 로봇 치수 정의 -->
   <xacro:property name="robot_length" value="0.86"/>
@@ -14,7 +24,5 @@
       </geometry>
       <origin xyz="0 0 0.05"/>
-      <material name="gray">
-        <color rgba="0.5 0.5 0.5 1"/>
-      </material>
+      <material name="gray"/>
     </visual>
     <collision>
@@ -30,4 +38,7 @@
     </inertial>
   </link>
+  <gazebo reference="base_link">
+    <material>Gazebo/White</material>
+  </gazebo>
   <!-- 바퀴 매크로 (회전 가능) -->
   <xacro:macro name="wheel" params="wheel_name wheel_joint x y z">
@@ -38,7 +49,5 @@
         </geometry>
         <origin rpy="-1.5708 0 0"/>
-        <material name="black">
-          <color rgba="0.2 0.2 0.2 1"/>
-        </material>
+        <material name="black"/>
       </visual>
       <collision>
@@ -55,6 +64,6 @@
             <friction>
               <ode>
-                <mu>1.0</mu>     <!-- 마찰 계수, 상황에 따라 1.0 ~ 2.0 등으로 조절 -->
-                <mu2>1.0</mu2>
+                <mu>0.6</mu>     <!-- 전진 마찰력 -->
+                <mu2>0.01</mu2>  <!-- 측면 마찰력(옴니 휠 적용) -->
               </ode>
             </friction>
@@ -81,30 +90,38 @@
                wheel_joint="front_left_wheel_joint"
                x="0.3" y="0.34" z="0"/>
+  <gazebo reference="front_left_wheel">
+    <material>Gazebo/BlackTransparent</material>
+  </gazebo>
   <xacro:wheel wheel_name="middle_left_wheel"
                wheel_joint="middle_left_wheel_joint"
                x="0.0" y="0.34" z="0"/>
+  <gazebo reference="middle_left_wheel">
+    <material>Gazebo/Black</material>
+  </gazebo>
   <xacro:wheel wheel_name="rear_left_wheel"
                wheel_joint="rear_left_wheel_joint"
                x="-0.3" y="0.34" z="0"/>
+  <gazebo reference="rear_left_wheel">
+    <material>Gazebo/BlackTransparent</material>
+  </gazebo>
   <xacro:wheel wheel_name="front_right_wheel"
                wheel_joint="front_right_wheel_joint"
                x="0.3" y="-0.34" z="0"/>
+  <gazebo reference="front_right_wheel">
+    <material>Gazebo/BlackTransparent</material>
+  </gazebo>
   <xacro:wheel wheel_name="middle_right_wheel"
                wheel_joint="middle_right_wheel_joint"
                x="0.0" y="-0.34" z="0"/>
+  <gazebo reference="middle_right_wheel">
+    <material>Gazebo/Black</material>
+  </gazebo>
   <xacro:wheel wheel_name="rear_right_wheel"
                wheel_joint="rear_right_wheel_joint"
                x="-0.3" y="-0.34" z="0"/>
+    <gazebo reference="rear_right_wheel">
+    <material>Gazebo/BlackTransparent</material>
+  </gazebo>
   <!-- Transmission (ros2_control) -->
-  <transmission name="front_left_trans">
-    <type>transmission_interface/SimpleTransmission</type>
-    <joint name="front_left_wheel_joint">
-      <interfaceType>hardware_interface/VelocityJointInterface</interfaceType>
-    </joint>
-    <actuator name="front_left_motor">
-      <mechanicalReduction>1</mechanicalReduction>
-      <hardwareInterface>hardware_interface/VelocityJointInterface</hardwareInterface>
-    </actuator>
-  </transmission>
   <transmission name="middle_left_trans">
     <type>transmission_interface/SimpleTransmission</type>
@@ -113,24 +130,4 @@
     </joint>
     <actuator name="middle_left_motor">
-      <mechanicalReduction>1</mechanicalReduction>
-      <hardwareInterface>hardware_interface/VelocityJointInterface</hardwareInterface>
-    </actuator>
-  </transmission>
-  <transmission name="rear_left_trans">
-    <type>transmission_interface/SimpleTransmission</type>
-    <joint name="rear_left_wheel_joint">
-      <interfaceType>hardware_interface/VelocityJointInterface</interfaceType>
-    </joint>
-    <actuator name="rear_left_motor">
-      <mechanicalReduction>1</mechanicalReduction>
-      <hardwareInterface>hardware_interface/VelocityJointInterface</hardwareInterface>
-    </actuator>
-  </transmission>
-  <transmission name="front_right_trans">
-    <type>transmission_interface/SimpleTransmission</type>
-    <joint name="front_right_wheel_joint">
-      <interfaceType>hardware_interface/VelocityJointInterface</interfaceType>
-    </joint>
-    <actuator name="front_right_motor">
       <mechanicalReduction>1</mechanicalReduction>
       <hardwareInterface>hardware_interface/VelocityJointInterface</hardwareInterface>
@@ -147,14 +144,4 @@
     </actuator>
   </transmission>
-  <transmission name="rear_right_trans">
-    <type>transmission_interface/SimpleTransmission</type>
-    <joint name="rear_right_wheel_joint">
-      <interfaceType>hardware_interface/VelocityJointInterface</interfaceType>
-    </joint>
-    <actuator name="rear_right_motor">
-      <mechanicalReduction>1</mechanicalReduction>
-      <hardwareInterface>hardware_interface/VelocityJointInterface</hardwareInterface>
-    </actuator>
-  </transmission>
   <!-- Lidar front -->
   <link name="lidar_front_link">
@@ -164,7 +151,5 @@
       </geometry>
       <origin xyz="0 0 0"/>
-      <material name="red">
-        <color rgba="1 0 0 1"/>
-      </material>
+      <material name="red"/>
     </visual>
   </link>
@@ -187,4 +172,7 @@
     </sensor>
   </gazebo>
+  <gazebo reference="lidar_front_link">
+    <material>Gazebo/Red</material>
+  </gazebo>
   <!-- Lidar rear -->
   <link name="lidar_rear_link">
@@ -193,7 +181,5 @@
         <cylinder length="0.04" radius="0.05"/>
       </geometry>
-      <material name="red">
-        <color rgba="0 1 0 1"/>
-      </material>
+      <material name="red"/>
     </visual>
   </link>
@@ -216,4 +202,7 @@
     </sensor>
   </gazebo>
+  <gazebo reference="lidar_rear_link">
+    <material>Gazebo/Red</material>
+  </gazebo>
   <ros2_control name="GazeboSystem" type="system">
     <hardware>
@@ -221,13 +210,4 @@
       <plugin>gazebo_ros2_control/GazeboSystem</plugin>
     </hardware>
-    <!-- 왼쪽 휠 조인트들 -->
-    <joint name="front_left_wheel_joint">
-      <command_interface name="velocity">
-        <param name="min">-1.0</param>
-        <param name="max">1.0</param>
-      </command_interface>
-      <state_interface name="position"/>
-      <state_interface name="velocity"/>
-    </joint>
     <joint name="middle_left_wheel_joint">
       <command_interface name="velocity">
@@ -238,21 +218,4 @@
       <state_interface name="velocity"/>
     </joint>
-    <joint name="rear_left_wheel_joint">
-      <command_interface name="velocity">
-        <param name="min">-1.0</param>
-        <param name="max">1.0</param>
-      </command_interface>
-      <state_interface name="position"/>
-      <state_interface name="velocity"/>
-    </joint>
-    <!-- 오른쪽 휠 조인트들 -->
-    <joint name="front_right_wheel_joint">
-      <command_interface name="velocity">
-        <param name="min">-1.0</param>
-        <param name="max">1.0</param>
-      </command_interface>
-      <state_interface name="position"/>
-      <state_interface name="velocity"/>
-    </joint>
     <joint name="middle_right_wheel_joint">
       <command_interface name="velocity">
@@ -263,12 +226,4 @@
       <state_interface name="velocity"/>
     </joint>
-    <joint name="rear_right_wheel_joint">
-      <command_interface name="velocity">
-        <param name="min">-1.0</param>
-        <param name="max">1.0</param>
-      </command_interface>
-      <state_interface name="position"/>
-      <state_interface name="velocity"/>
-    </joint>
   </ros2_control>
   <!-- gazebo_ros2_control plugin -->

Commit message: update

File: install/my_robot_description/share/my_robot_description/urdf/amr_robot.urdf.xacro (robot description, xacro)
@@ -41,5 +41,5 @@
     <material>Gazebo/White</material>
   </gazebo>
-  <!-- 바퀴 매크로 (회전 가능) -->
+  <!-- 바퀴 매크로 (실제 구동) -->
   <xacro:macro name="wheel" params="wheel_name wheel_joint x y z">
     <link name="${wheel_name}">
@@ -56,14 +56,12 @@
         </geometry>
         <origin rpy="-1.5708 0 0"/>
-        <!--
-          바퀴와 지면 사이의 마찰을 적용하기 위해
-          Gazebo SDF 확장 태그(material > friction > ode > mu/mu2) 추가
-        -->
         <gazebo>
           <material>
             <friction>
               <ode>
-                <mu>0.6</mu>     <!-- 전진 마찰력 -->
-                <mu2>0.01</mu2>  <!-- 측면 마찰력(옴니 휠 적용) -->
+                <mu>0.8</mu>     <!-- 전진 마찰력 -->
+                <mu2>0.05</mu2>  <!-- 측면 마찰력 -->
+                <slip1>0.5</slip1>  <!-- 약간의 슬립 적용 (너무 높으면 미끄러짐) -->
+                <slip2>0.5</slip2>
               </ode>
             </friction>
@@ -86,6 +84,49 @@
     </joint>
   </xacro:macro>
+  <!-- 바퀴 매크로 (옴니 휠, 실제 구동X) -->
+  <xacro:macro name="omni_wheel" params="wheel_name wheel_joint x y z">
+    <link name="${wheel_name}">
+      <visual>
+        <geometry>
+          <cylinder length="${wheel_thickness}" radius="${wheel_radius}"/>
+        </geometry>
+        <origin rpy="-1.5708 0 0"/>
+        <material name="black"/>
+      </visual>
+      <collision>
+       <geometry>
+        <cylinder length="${wheel_thickness}" radius="${wheel_radius}"/>
+       </geometry>
+       <origin rpy="-1.5708 0 0"/>
+        <gazebo>
+          <material>
+            <friction>
+              <ode>
+                <mu>0.6</mu>        <!-- 전진 마찰력 -->
+                <mu2>0.01</mu2>      <!-- 측면 마찰력(낮게 설정) -->
+                <slip1>2.0</slip1>    <!-- 전방 슬립 파라미터 -->
+                <slip2>2.0</slip2>    <!-- 측면 슬립 파라미터 -->
+              </ode>
+            </friction>
+          </material>
+        </gazebo>
+      </collision>
+    <inertial>
+      <mass value="2"/>
+      <origin xyz="0 0 0"/>
+      <inertia ixx="0.01225" ixy="0" ixz="0" iyy="0.01225" iyz="0" izz="0.0093"/>
+    </inertial>
+  </link>
+  <joint name="${wheel_joint}" type="continuous">
+    <parent link="base_link"/>
+    <child link="${wheel_name}"/>
+    <origin xyz="${x} ${y} ${z}"/>
+    <axis xyz="0 1 0"/>
+    <limit effort="30" velocity="10"/>
+    <dynamics damping="1.0" friction="0.2"/>
+  </joint>
+</xacro:macro>
   <!-- 6개 바퀴 정의 -->
-  <xacro:wheel wheel_name="front_left_wheel"
+  <xacro:omni_wheel wheel_name="front_left_wheel"
                wheel_joint="front_left_wheel_joint"
                x="0.3" y="0.34" z="0"/>
@@ -99,5 +140,5 @@
     <material>Gazebo/Black</material>
   </gazebo>
-  <xacro:wheel wheel_name="rear_left_wheel"
+  <xacro:omni_wheel wheel_name="rear_left_wheel"
                wheel_joint="rear_left_wheel_joint"
                x="-0.3" y="0.34" z="0"/>
@@ -105,5 +146,5 @@
     <material>Gazebo/BlackTransparent</material>
   </gazebo>
-  <xacro:wheel wheel_name="front_right_wheel"
+  <xacro:omni_wheel wheel_name="front_right_wheel"
                wheel_joint="front_right_wheel_joint"
                x="0.3" y="-0.34" z="0"/>
@@ -117,5 +158,5 @@
     <material>Gazebo/Black</material>
   </gazebo>
-  <xacro:wheel wheel_name="rear_right_wheel"
+  <xacro:omni_wheel wheel_name="rear_right_wheel"
                wheel_joint="rear_right_wheel_joint"
                x="-0.3" y="-0.34" z="0"/>
